File: scast_goad.kicad_sch (KiCad schematic)
At the start: 15 parts, among them SW1 SW_Push, SW2 RotaryEncoder_Switch, SW5 SW_Push, SW6 SW_Push, U1 ESP32-S3-WROOM-1

Commit message: Finished first schematic iteration and added footprints
Parts:
- removed C1, C2, C3: C_Small, symbol Device:C_Small
- removed R1, R2: R_Small, symbol Device:R_Small
- removed SW1: SW_Push, symbol Switch:SW_Push
- removed SW2: RotaryEncoder_Switch, symbol Device:RotaryEncoder_Switch
- removed U1: ESP32-S3-WROOM-1, RF_Module:ESP32-S3-WROOM-1, symbol RF_Module:ESP32-S3-WROOM-1
- added A1: Arduino_UNO_R3, Module:Arduino_UNO_R3, symbol MCU_Module:Arduino_UNO_R3
- added J1: Rotary Encoder, Connector_PinSocket_2.54mm:PinSocket_1x05_P2.54mm_Horizontal, symbol Connector:Conn_01x05_Socket
- added J2: Tilt_Sensor, Connector_PinSocket_2.54mm:PinSocket_1x06_P2.54mm_Horizontal, symbol Connector:Conn_01x06_Socket
- added TP1: TP_GND, TestPoint:TestPoint_Pad_D4.0mm, symbol Connector:TestPoint
- added TP2: TP_3V3, TestPoint:TestPoint_Pad_4.0x4.0mm, symbol Connector:TestPoint
- C4, C5: value C_Small -> C_Filter; footprint (none) -> Capacitor_THT:C_Disc_D11.0mm_W5.0mm_P10.00mm
- R3, R5, R6: value R_Small -> R_Pulldown; footprint (none) -> Resistor_THT:R_Axial_DIN0414_L11.9mm_D4.5mm_P15.24mm_Horizontal
- SW5, SW6: footprint (none) -> scatno2:SW_SANWA
Connections:
- net +3V3: now also A1.4 (3V3), J1.4 (Pin_4), J2.2 (Pin_2), TP2.1
- net BWD_SW: now also A1.19 (D4)
- net ENCODER_A: now also A1.17 (D2), J1.1 (Pin_1); no longer R3.1
- net ENCODER_B: now also A1.18 (D3), J1.2 (Pin_2)
- net FWD_SW: now also A1.20 (D5)
- net GND: now also A1.29 (GND), A1.6 (GND), A1.7 (GND), J2.1 (Pin_1), TP1.1
- new net: J1.5 (Pin_5), R3.1
- new net TILT_SCL: A1.14 (SCL/A5), J2.4 (Pin_4)
- new net TILT_SDA: A1.13 (SDA/A4), J2.3 (Pin_3)
- no-connect marks 0 -> 3
Other:
- note added: "Connectors"
- note added: "Motherboard (with integrated buttons)"
- moved on the sheet: C4, C5, R3, R5, R6, SW5, SW6

Commit message: Created Gerber Files for PCB
Parts:
- removed R3: R_Pulldown, Resistor_THT:R_Axial_DIN0414_L11.9mm_D4.5mm_P15.24mm_Horizontal, symbol Device:R_Small
Connections:
- net GND: now also J1.5 (Pin_5)
- no-connect marks 3 -> 24
Changed lines of the file:
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@@
+	)
+	(no_connect
+		(at 60.96 68.58)
+	)
+	(no_connect
+		(at 60.96 53.34)
+	)
+	(no_connect
+		(at 35.56 38.1)
+	)
+	(no_connect
+		(at 35.56 55.88)
+	)
+	(no_connect
+		(at 60.96 50.8)
+	)
+	(no_connect
+		(at 60.96 45.72)
+	)
+	(no_connect
+		(at 45.72 25.4)
+	)
+	(no_connect
+		(at 53.34 25.4)
+	)
+	(no_connect
+		(at 35.56 66.04)
+	)
+	(no_connect
+		(at 60.96 55.88)
+	)
+	(no_connect
+		(at 35.56 53.34)
+	)
+	(no_connect
+		(at 60.96 58.42)
+	)
+	(no_connect
+		(at 35.56 68.58)
+	)
+	(no_connect
+		(at 35.56 35.56)
+	)
+	(no_connect
+		(at 60.96 35.56)
+	)
+	(no_connect
+		(at 35.56 60.96)
+	)
+	(no_connect
+		(at 35.56 50.8)
 	)
 	(no_connect
@@
 		(at 123.19 34.29)
 	)
+	(no_connect
+		(at 35.56 58.42)
+	)
+	(no_connect
+		(at 60.96 71.12)
+	)
+	(no_connect
+		(at 35.56 63.5)
+	)
+	(no_connect
+		(at 60.96 40.64)
+	)
 	(wire
 		(pts
@@
 	(wire
 		(pts
+			(xy 124.46 41.91) (xy 124.46 39.37)
+		)
+		(stroke
+			(width 0)
+			(type default)
+		)
+	)
+	(wire
+		(pts
 			(xy 62.23 60.96) (xy 60.96 60.96)
 		)
@@
 	(wire
 		(pts
+			(xy 85.09 60.96) (xy 85.09 59.69)
+		)
+		(stroke
+			(width 0)
+			(type default)
+		)
+	)
+	(wire
+		(pts
+			(xy 125.73 81.28) (xy 125.73 78.74)
+		)
+		(stroke
+			(width 0)
+			(type default)
+		)
+	)
+	(wire
+		(pts
+			(xy 33.02 48.26) (xy 35.56 48.26)
+		)
+		(stroke
+			(width 0)
+			(type default)
+		)
+	)
+	(wire
+		(pts
+			(xy 123.19 36.83) (xy 127 36.83)
+		)
+		(stroke
+			(width 0)
+			(type default)
+		)
+	)
+	(wire
+		(pts
+			(xy 90.17 63.5) (xy 90.17 60.96)
+		)
+		(stroke
+			(width 0)
+			(type default)
+		)
+	)
+	(wire
+		(pts
+			(xy 85.09 36.83) (xy 85.09 38.1)
+		)
+		(stroke
+			(width 0)
+			(type default)
+		)
+	)
+	(wire
+		(pts
+			(xy 48.26 78.74) (xy 45.72 78.74)
+		)
+		(stroke
+			(width 0)
+			(type default)
+		)
+	)
+	(wire
+		(pts
+			(xy 85.09 36.83) (xy 90.17 36.83)
+		)
+		(stroke
+			(width 0)
+			(type default)
+		)
+	)
+	(wire
+		(pts
+			(xy 90.17 34.29) (xy 90.17 36.83)
+		)
+		(stroke
+			(width 0)
+			(type default)
+		)
+	)
+	(wire
+		(pts
 			(xy 124.46 39.37) (xy 123.19 39.37)
-		)
-		(stroke
-			(width 0)
-			(type default)
-		)
-	)
-	(wire
-		(pts
-			(xy 85.09 60.96) (xy 85.09 59.69)
-		)
-		(stroke
-			(width 0)
-			(type default)
-		)
-	)
-	(wire
-		(pts
-			(xy 124.46 44.45) (xy 124.46 45.72)
-		)
-		(stroke
-			(width 0)
-			(type default)
-		)
-	)
-	(wire
-		(pts
-			(xy 125.73 81.28) (xy 125.73 78.74)
-		)
-		(stroke
-			(width 0)
-			(type default)
-		)
-	)
-	(wire
-		(pts
-			(xy 33.02 48.26) (xy 35.56 48.26)
-		)
-		(stroke
-			(width 0)
-			(type default)
-		)
-	)
-	(wire
-		(pts
-			(xy 123.19 36.83) (xy 127 36.83)
-		)
-		(stroke
-			(width 0)
-			(type default)
-		)
-	)
-	(wire
-		(pts
-			(xy 90.17 63.5) (xy 90.17 60.96)
-		)
-		(stroke
-			(width 0)
-			(type default)
-		)
-	)
-	(wire
-		(pts
-			(xy 85.09 36.83) (xy 85.09 38.1)
-		)
-		(stroke
-			(width 0)
-			(type default)
-		)
-	)
-	(wire
-		(pts
-			(xy 48.26 78.74) (xy 45.72 78.74)
-		)
-		(stroke
-			(width 0)
-			(type default)
-		)
-	)
-	(wire
-		(pts
-			(xy 85.09 36.83) (xy 90.17 36.83)
-		)
-		(stroke
-			(width 0)
-			(type default)
-		)
-	)
-	(wire
-		(pts
-			(xy 90.17 34.29) (xy 90.17 36.83)
 		)
 		(stroke
@@
 		(property "Value" "TP_GND"
 			(at 25.4 79.2479 0)
-			(show_name no)
+			(show_name yes)
 			(do_not_autoplace no)
 			(effects
@@
 		(property "Value" "TP_3V3"
 			(at 25.4 71.8819 0)
-			(show_name no)
+			(show_name yes)
 			(do_not_autoplace no)
 			(effects
@@
 	(symbol
 		(lib_id "power:GND")
-		(at 124.46 45.72 0)
+		(at 124.46 41.91 0)
 		(mirror y)
 		(unit 1)
@@
 		(fields_autoplaced yes)
 		(property "Reference" "#PWR08"
-			(at 124.46 52.07 0)
+			(at 124.46 48.26 0)
 			(hide yes)
 			(show_name no)
@@
 		)
 		(property "Value" "GND"
-			(at 124.46 50.8 0)
+			(at 124.46 46.99 0)
 			(show_name no)
 			(do_not_autoplace no)
@@
 		)
 		(property "Footprint" ""
-			(at 124.46 45.72 0)
+			(at 124.46 41.91 0)
 			(hide yes)
 			(show_name no)
@@
 		)
 		(property "Datasheet" ""
-			(at 124.46 45.72 0)
+			(at 124.46 41.91 0)
 			(hide yes)
 			(show_name no)
@@
 		)
 		(property "Description" "Power symbol creates a global label with name \"GND\" , ground"
-			(at 124.46 45.72 0)
+			(at 124.46 41.91 0)
 			(hide yes)
 			(show_name no)
@@
 					(unit 1)
 				)
-			)
-		)
-	)
-	(symbol
-		(lib_id "Device:R_Small")
-		(at 124.46 41.91 0)
-		(mirror y)
-		(unit 1)
-		(body_style 1)
-		(exclude_from_sim no)
-		(in_bom yes)
-		(on_board yes)
-		(in_pos_files yes)
-		(dnp no)
-		(property "Reference" "R3"
-			(at 122.936 40.64 0)
-			(show_name no)
-			(do_not_autoplace no)
-			(effects
-				(font
-					(size 1.016 1.016)
-				)
-				(justify left)
-			)
-		)
-		(property "Value" "R_Pulldown"
-			(at 122.936 43.18 0)
-			(show_name no)
-			(do_not_autoplace no)
-			(effects
-				(font
-					(size 1.27 1.27)
-				)
-				(justify left)
-			)
-		)
-		(property "Footprint" "Resistor_THT:R_Axial_DIN0414_L11.9mm_D4.5mm_P15.24mm_Horizontal"
-			(at 124.46 41.91 0)
-			(hide yes)
-			(show_name no)
-			(do_not_autoplace no)
-			(effects
-				(font
-					(size 1.27 1.27)
-				)
-			)
-		)
-		(property "Datasheet" ""
-			(at 124.46 41.91 0)
-			(hide yes)
-			(show_name no)
-			(do_not_autoplace no)
-			(effects
-				(font
-					(size 1.27 1.27)
-				)
-			)
-		)
-		(property "Description" "Resistor, small symbol"
-			(at 124.46 41.91 0)
-			(hide yes)
-			(show_name no)
-			(do_not_autoplace no)
-			(effects
-				(font
-					(size 1.27 1.27)
-				)
-			)
-		)
-		(pin "2"
-		)
-		(pin "1"
-		)
-		(instances
-			(project "scast_goad"
-				(path "/e67bcb6b-497c-4fce-bafc-767002b94006"
-					(reference "R3")
-					(unit 1)
-				)
